File: Homework/Hw15/ME433 HW15/ME433 HW15.kicad_sch (KiCad schematic)
At the start: 11 parts, among them J1 Conn_01x03_Pin

Commit message: Hw #15 completed
Parts:
- C1, C2: footprint (none) -> Capacitor_SMD:C_0805_2012Metric
- D1: renamed from D2; footprint (none) -> Diode_SMD:D_SOD-123
- D2: renamed from D1; footprint (none) -> LED_SMD:LED_0603_1608Metric
- J1: footprint (none) -> Connector_PinHeader_2.54mm:PinHeader_1x03_P2.54mm_Vertical
- L1: footprint (none) -> Inductor_SMD:L_0603_1608Metric
- R1, R4: footprint (none) -> Resistor_SMD:R_0603_1608Metric
- R2, R3: footprint (none) -> Resistor_SMD:R_0402_1005Metric
- U1: footprint MT3608L -> Package_TO_SOT_SMD:TSOT-23-6_HandSoldering
Changed lines of the file:
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@@
 			)
 		)
-		(property "Footprint" ""
+		(property "Footprint" "Capacitor_SMD:C_0805_2012Metric"
 			(at 116.5352 97.79 0)
 			(effects
@@
 			)
 		)
-		(property "Footprint" ""
+		(property "Footprint" "Resistor_SMD:R_0603_1608Metric"
 			(at 150.114 96.774 90)
 			(effects
@@
 		(dnp no)
 		(fields_autoplaced yes)
-		(property "Reference" "#PWR012"
+		(property "Reference" "#PWR014"
 			(at 191.77 73.66 0)
 			(effects
@@
 			(project ""
 				(path "/1471c6a4-b32d-4f8e-8c73-db65409b2a6b"
-					(reference "#PWR012")
+					(reference "#PWR014")
 					(unit 1)
 				)
@@
 		(dnp no)
 		(fields_autoplaced yes)
-		(property "Reference" "#PWR07"
+		(property "Reference" "#PWR01"
 			(at 73.66 96.52 0)
 			(effects
@@
 			(project ""
 				(path "/1471c6a4-b32d-4f8e-8c73-db65409b2a6b"
-					(reference "#PWR07")
+					(reference "#PWR01")
 					(unit 1)
 				)
@@
 		(dnp no)
 		(fields_autoplaced yes)
-		(property "Reference" "#PWR04"
+		(property "Reference" "#PWR011"
 			(at 170.18 115.57 0)
 			(effects
@@
 			(project ""
 				(path "/1471c6a4-b32d-4f8e-8c73-db65409b2a6b"
-					(reference "#PWR04")
+					(reference "#PWR011")
 					(unit 1)
 				)
@@
 			)
 		)
-		(property "Footprint" ""
+		(property "Footprint" "Capacitor_SMD:C_0805_2012Metric"
 			(at 98.7552 97.79 0)
 			(effects
@@
 		(dnp no)
 		(fields_autoplaced yes)
-		(property "Reference" "#PWR011"
+		(property "Reference" "#PWR010"
 			(at 165.1 73.66 0)
 			(effects
@@
 			(project ""
 				(path "/1471c6a4-b32d-4f8e-8c73-db65409b2a6b"
-					(reference "#PWR011")
+					(reference "#PWR010")
 					(unit 1)
 				)
@@
 		(on_board yes)
 		(dnp no)
-		(property "Reference" "D2"
+		(property "Reference" "D1"
 			(at 172.4025 68.58 0)
 			(effects
@@
 			)
 		)
-		(property "Footprint" ""
+		(property "Footprint" "Diode_SMD:D_SOD-123"
 			(at 172.72 74.93 0)
 			(effects
@@
 			(project ""
 				(path "/1471c6a4-b32d-4f8e-8c73-db65409b2a6b"
-					(reference "D2")
+					(reference "D1")
 					(unit 1)
 				)
@@
 		(dnp no)
 		(fields_autoplaced yes)
-		(property "Reference" "#PWR016"
+		(property "Reference" "#PWR015"
 			(at 223.52 85.09 0)
 			(effects
@@
 			(project ""
 				(path "/1471c6a4-b32d-4f8e-8c73-db65409b2a6b"
-					(reference "#PWR016")
+					(reference "#PWR015")
 					(unit 1)
 				)
@@
 		(dnp no)
 		(fields_autoplaced yes)
-		(property "Reference" "#PWR01"
+		(property "Reference" "#PWR03"
 			(at 80.01 106.68 0)
 			(effects
@@
 			(project ""
 				(path "/1471c6a4-b32d-4f8e-8c73-db65409b2a6b"
-					(reference "#PWR01")
+					(reference "#PWR03")
 					(unit 1)
 				)
@@
 			)
 		)
-		(property "Footprint" "MT3608L"
+		(property "Footprint" "Package_TO_SOT_SMD:TSOT-23-6_HandSoldering"
 			(at 170.434 86.36 0)
 			(effects
@@
 		(dnp no)
 		(fields_autoplaced yes)
-		(property "Reference" "#PWR08"
+		(property "Reference" "#PWR04"
 			(at 97.79 90.17 0)
 			(effects
@@
 			(project ""
 				(path "/1471c6a4-b32d-4f8e-8c73-db65409b2a6b"
-					(reference "#PWR08")
+					(reference "#PWR04")
 					(unit 1)
 				)
@@
 			)
 		)
-		(property "Footprint" ""
+		(property "Footprint" "Resistor_SMD:R_0402_1005Metric"
 			(at 187.706 104.394 90)
 			(effects
@@
 		(dnp no)
 		(fields_autoplaced yes)
-		(property "Reference" "#PWR015"
+		(property "Reference" "#PWR016"
 			(at 223.52 111.76 0)
 			(effects
@@
 			(project ""
 				(path "/1471c6a4-b32d-4f8e-8c73-db65409b2a6b"
-					(reference "#PWR015")
+					(reference "#PWR016")
 					(unit 1)
 				)
@@
 		(dnp no)
 		(fields_autoplaced yes)
-		(property "Reference" "#PWR013"
+		(property "Reference" "#PWR012"
 			(at 186.69 88.9 0)
 			(effects
@@
 			(project ""
 				(path "/1471c6a4-b32d-4f8e-8c73-db65409b2a6b"
-					(reference "#PWR013")
+					(reference "#PWR012")
 					(unit 1)
 				)
@@
 		(dnp no)
 		(fields_autoplaced yes)
-		(property "Reference" "#PWR06"
+		(property "Reference" "#PWR02"
 			(at 80.01 90.17 0)
 			(effects
@@
 			(project ""
 				(path "/1471c6a4-b32d-4f8e-8c73-db65409b2a6b"
-					(reference "#PWR06")
+					(reference "#PWR02")
 					(unit 1)
 				)
@@
 		(dnp no)
 		(fields_autoplaced yes)
-		(property "Reference" "D1"
+		(property "Reference" "D2"
 			(at 227.33 87.9474 90)
 			(effects
@@
 			)
 		)
-		(property "Footprint" ""
+		(property "Footprint" "LED_SMD:LED_0603_1608Metric"
 			(at 223.52 87.63 0)
 			(effects
@@
 			(project ""
 				(path "/1471c6a4-b32d-4f8e-8c73-db65409b2a6b"
-					(reference "D1")
+					(reference "D2")
 					(unit 1)
 				)
@@
 			)
 		)
-		(property "Footprint" ""
+		(property "Footprint" "Resistor_SMD:R_0603_1608Metric"
 			(at 224.536 99.314 90)
 			(effects
@@
 		(dnp no)
 		(fields_autoplaced yes)
-		(property "Reference" "#PWR010"
+		(property "Reference" "#PWR09"
 			(at 156.21 87.63 0)
 			(effects
@@
 			(project ""
 				(path "/1471c6a4-b32d-4f8e-8c73-db65409b2a6b"
-					(reference "#PWR010")
+					(reference "#PWR09")
 					(unit 1)
 				)
@@
 		(dnp no)
 		(fields_autoplaced yes)
-		(property "Reference" "#PWR03"
+		(property "Reference" "#PWR07"
 			(at 115.57 107.95 0)
 			(effects
@@
 			(project ""
 				(path "/1471c6a4-b32d-4f8e-8c73-db65409b2a6b"
-					(reference "#PWR03")
+					(reference "#PWR07")
 					(unit 1)
 				)
@@
 			)
 		)
-		(property "Footprint" ""
+		(property "Footprint" "Resistor_SMD:R_0402_1005Metric"
 			(at 187.706 91.694 90)
 			(effects
@@
 		(dnp no)
 		(fields_autoplaced yes)
-		(property "Reference" "#PWR02"
+		(property "Reference" "#PWR05"
 			(at 97.79 107.95 0)
 			(effects
@@
 			(project ""
 				(path "/1471c6a4-b32d-4f8e-8c73-db65409b2a6b"
-					(reference "#PWR02")
+					(reference "#PWR05")
 					(unit 1)
 				)
@@
 			)
 		)
-		(property "Footprint" ""
+		(property "Footprint" "Inductor_SMD:L_0603_1608Metric"
 			(at 185.42 74.93 0)
 			(effects
@@
 		(dnp no)
 		(fields_autoplaced yes)
-		(property "Reference" "#PWR05"
+		(property "Reference" "#PWR08"
 			(at 144.78 107.95 0)
 			(effects
@@
 			(project ""
 				(path "/1471c6a4-b32d-4f8e-8c73-db65409b2a6b"
-					(reference "#PWR05")
+					(reference "#PWR08")
 					(unit 1)
 				)
@@
 		(dnp no)
 		(fields_autoplaced yes)
-		(property "Reference" "#PWR014"
+		(property "Reference" "#PWR013"
 			(at 186.69 116.84 0)
 			(effects
@@
 			(project ""
 				(path "/1471c6a4-b32d-4f8e-8c73-db65409b2a6b"
-					(reference "#PWR014")
+					(reference "#PWR013")
 					(unit 1)
 				)
@@
 		(dnp no)
 		(fields_autoplaced yes)
-		(property "Reference" "#PWR09"
+		(property "Reference" "#PWR06"
 			(at 115.57 90.17 0)
 			(effects
@@
 			(project ""
 				(path "/1471c6a4-b32d-4f8e-8c73-db65409b2a6b"
-					(reference "#PWR09")
+					(reference "#PWR06")
 					(unit 1)
 				)
@@
 			)
 		)
-		(property "Footprint" ""
+		(property "Footprint" "Connector_PinHeader_2.54mm:PinHeader_1x03_P2.54mm_Vertical"
 			(at 66.04 95.25 0)
 			(effects
